File: mkii.brd (EAGLE design)
At the start: 47.8 x 29 mm, 52 parts, among them IC1 ATMEGA32U4, Q1 16MHz, U1 GTL2003, U2 TS1117, U3 PRTR5V0U2AX, X1 MINI-USB-32005-301

Commit message: atmega32u2, not u4
Parts:
- IC1: value ATMEGA32U4 -> ATMEGA32U2
Changed lines of the file:
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@@
 </autorouter>
 <elements>
-<element name="IC1" library="at90usb" package="TQFP32-08" value="ATMEGA32U4" x="16.51" y="8.89" smashed="yes" rot="MR270">
+<element name="IC1" library="at90usb" package="TQFP32-08" value="ATMEGA32U2" x="16.51" y="8.89" smashed="yes" rot="MR270">
 <attribute name="NAME" x="22.1996" y="4.191" size="1.016" layer="26" rot="MR0"/>
 <attribute name="VALUE" x="17.78" y="11.9126" size="0.8128" layer="28" rot="MR270"/>
@@
 </signal>
 </signals>
-<errors>
-</errors>
 </board>
 </drawing>
